File: 26th_PCB_PitchSender.kicad_pcb (KiCad board)
At the start: 2 copper layers, 120 x 28.4 mm, 16 parts, among them J1 Amp, J2 Conn_01x04_Pin, J3 microSD, J4 BNO055, J5 Conn_01x04_Socket, U1 ESP32-DEVKITC-32E

Commit message: 一応完成
Parts:
- moved H1 0.38 mm to (217.8, 79.8)
- moved H2 0.27 mm to (217.8, 101.1)
Routing:
- net Net-(J1-Pin_2): track 0.00 -> 122.1 mm
- net GND: track 80.0 -> 181.0 mm, vias 2 -> 3
- net +5V: track 16.8 -> 114.9 mm, vias 0 -> 4
- net /BicoRX-psdTX: track 0.00 -> 80.6 mm
- net /BicoTX-psdRX: track 0.00 -> 71.7 mm
- net /ChipSelect: track 0.00 -> 51.9 mm
- net /SPK: track 0.00 -> 51.9 mm, vias 0 -> 2
- net +3V3: track 0.00 -> 47.2 mm
- net /MISO: track 0.00 -> 32.9 mm
- net /SCL: track 0.00 -> 32.1 mm, vias 0 -> 3
- net /SCK: track 0.00 -> 27.4 mm, vias 0 -> 1
- net /MOSI: track 0.00 -> 25.2 mm, vias 0 -> 1
- net /SDA: track 0.00 -> 24.2 mm, vias 0 -> 2
Other:
- outline, holes or cut-outs redrawn

Commit message: BMP追加
Parts:
- added D2: LED, LED_THT:LED_D3.0mm, F.Cu at (211.8, 101.5)
- added D3: LED, LED_THT:LED_D3.0mm, F.Cu at (211.0, 79.2)
- added J6: BMP390, Connector_PinHeader_2.54mm:PinHeader_1x04_P2.54mm_Vertical, B.Cu at (127.2, 83.5)
- added R2: R, Resistor_THT:R_Axial_DIN0204_L3.6mm_D1.6mm_P5.08mm_Horizontal, F.Cu at (192.0, 101.8)
- added R3: R, Resistor_THT:R_Axial_DIN0204_L3.6mm_D1.6mm_P5.08mm_Horizontal, F.Cu at (193.0, 79.2)
- J1: value Amp -> vol
- J4: value BNO055 -> Conn_01x04_Socket
- J5: value Conn_01x04_Socket -> BNO055
- RV1: value Vol -> vol
- U1: value ESP32-DEVKITC-32E -> ~
Connections:
- U1 pad J3_13: unconnected-(U1-IO4-PadJ3_13) -> Net-(U1-IO4)
- U1 pad J3_16: unconnected-(U1-IO15-PadJ3_16) -> Net-(U1-IO15)
Routing:
- net GND: track 181.0 -> 243.4 mm
- net Net-(U1-IO4): track 0.00 -> 33.7 mm
- net +3V3: track 47.2 -> 76.2 mm
- net /SDA: track 24.2 -> 52.8 mm
- net Net-(J1-Pin_2): track 122.1 -> 95.1 mm, vias 0 -> 2
- net /SCL: track 32.1 -> 53.6 mm, vias 3 -> 4
- net Net-(U1-IO15): track 0.00 -> 17.3 mm
- net Net-(D2-A): track 0.00 -> 12.3 mm
- net Net-(D3-A): track 0.00 -> 10.4 mm
- net +5V: track 114.9 -> 109.7 mm, vias 4 -> 6
