File: 26th_PCB_PitchSender.kicad_pcb (KiCad board)
At the start: 2 copper layers, 120.2 x 28.5 mm, 21 parts, among them J1 Amp, J2 Conn_01x04_Pin, J3 microSD, J4 BNO055, J5 BNO055, J6 BMP390

Commit message: Add PA connecter
Parts:
- added JP1: S03B-PASK-2, lib:S03B-PASK-2, F.Cu at (120.8, 95.8)
- moved R1 3.69 mm to (119.2, 85.6)
Routing:
- net /SPK: track 101.2 -> 119.9 mm
- net Net-(J1-Pin_2): track 45.3 -> 49.9 mm
- net +5V: track 123.9 -> 120.6 mm
- net GND: track 169.4 -> 167.1 mm, vias 2 -> 0
- net Net-(D1-A): track 4.30 -> 5.39 mm
Other:
- outline, holes or cut-outs redrawn
