File: 26th_PCB_PitchSender.kicad_pcb (KiCad board)
At the start: 2 copper layers, 120.2 x 28.5 mm, 22 parts, among them J1 Amp, J2 Conn_01x04_Pin, J3 microSD, J4 BNO055, J5 BNO055, J6 BMP390

Commit message: Change SPK pin
Parts:
- J4: value BNO055 -> Conn_01x04_Socket
Connections:
- U1 pad J2_15: unconnected-(U1-IO13-PadJ2_15) -> /SPK
- U1 pad J3_11: /SPK -> unconnected-(U1-IO17-PadJ3_11)
Routing:
- net /SPK: track 111.8 -> 91.7 mm, vias 3 -> 2
Changed lines of the file:
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@@
 	(net 44 "unconnected-(U1-IO14-PadJ2_12)")
 	(net 45 "unconnected-(U1-IO12-PadJ2_13)")
-	(net 46 "unconnected-(U1-IO13-PadJ2_15)")
+	(net 46 "unconnected-(U1-IO17-PadJ3_11)")
 	(net 47 "Net-(U1-IO4)")
 	(net 48 "unconnected-(U1-RXD0-PadJ3_5)")
@@
 			(layers "*.Cu" "*.Mask")
 			(remove_unused_layers no)
-			(net 46 "unconnected-(U1-IO13-PadJ2_15)")
+			(net 12 "/SPK")
 			(pinfunction "IO13")
-			(pintype "bidirectional+no_connect")
+			(pintype "bidirectional")
 			(solder_mask_margin 0.102)
 		)
@@
 			(layers "*.Cu" "*.Mask")
 			(remove_unused_layers no)
-			(net 12 "/SPK")
+			(net 46 "unconnected-(U1-IO17-PadJ3_11)")
 			(pinfunction "IO17")
-			(pintype "bidirectional")
+			(pintype "bidirectional+no_connect")
 			(solder_mask_margin 0.102)
 		)
@@
 			)
 		)
-		(property "Value" "BNO055"
+		(property "Value" "Conn_01x04_Socket"
 			(at 4.1 -10.82 90)
 			(layer "B.SilkS")
@@
 	)
 	(segment
-		(start 180 97.25)
-		(end 197.8189 97.25)
+		(start 123.931 102.29)
+		(end 123.391 101.75)
 		(width 0.2)
 		(layer "F.Cu")
@@
 	)
 	(segment
-		(start 155.075 103.5)
-		(end 161.5 103.5)
+		(start 182.75 100.5)
+		(end 182.54 100.29)
 		(width 0.2)
 		(layer "F.Cu")
@@
 	)
 	(segment
-		(start 136.75 101.75)
-		(end 153.325 101.75)
+		(start 202.09 103.44)
+		(end 200.75 102.1)
 		(width 0.2)
 		(layer "F.Cu")
@@
 	)
 	(segment
-		(start 135.75 101.75)
-		(end 136.75 101.75)
+		(start 158.46 102.29)
+		(end 123.931 102.29)
 		(width 0.2)
 		(layer "F.Cu")
@@
 	)
 	(segment
-		(start 161.5 103.5)
-		(end 164.25 100.75)
+		(start 182.54 100.29)
+		(end 160.46 100.29)
 		(width 0.2)
 		(layer "F.Cu")
@@
 	)
 	(segment
-		(start 131.5 101.75)
-		(end 135.75 101.75)
+		(start 160.46 100.29)
+		(end 158.46 102.29)
 		(width 0.2)
 		(layer "F.Cu")
@@
 	)
 	(segment
-		(start 153.325 101.75)
-		(end 155.075 103.5)
+		(start 200.75 102.1)
+		(end 188.25 102.1)
 		(width 0.2)
 		(layer "F.Cu")
 		(net 12)
 	)
-	(segment
-		(start 197.8189 97.25)
-		(end 199.7478 95.3211)
-		(width 0.2)
-		(layer "F.Cu")
-		(net 12)
-	)
-	(segment
-		(start 123.391 101.75)
-		(end 131.5 101.75)
-		(width 0.2)
-		(layer "F.Cu")
-		(net 12)
-	)
-	(segment
-		(start 175.75 100.75)
-		(end 177.25 99.25)
-		(width 0.2)
-		(layer "F.Cu")
-		(net 12)
-	)
-	(segment
-		(start 164.25 100.75)
-		(end 175.75 100.75)
-		(width 0.2)
-		(layer "F.Cu")
-		(net 12)
-	)
-	(via
-		(at 180 97.25)
-		(size 0.6)
-		(drill 0.3)
-		(layers "F.Cu" "B.Cu")
-		(net 12)
-	)
 	(via
-		(at 199.7478 95.3211)
+		(at 188.25 102.1)
 		(size 0.6)
 		(drill 0.3)
@@
 	)
 	(via
-		(at 177.25 99.25)
+		(at 182.75 100.5)
 		(size 0.6)
 		(drill 0.3)
@@
 	)
 	(segment
-		(start 199.7478 90.6528)
-		(end 191.7227 82.6277)
-		(width 0.2)
-		(layer "B.Cu")
-		(net 12)
-	)
-	(segment
-		(start 191.7227 78.2473)
-		(end 191.93 78.04)
-		(width 0.2)
-		(layer "B.Cu")
-		(net 12)
-	)
-	(segment
-		(start 199.7478 95.3211)
-		(end 199.7478 90.6528)
+		(start 188.25 102.1)
+		(end 184.35 102.1)
 		(width 0.2)
 		(layer "B.Cu")
@@
 	)
 	(segment
-		(start 179.25 97.25)
-		(end 180 97.25)
-		(width 0.2)
-		(layer "B.Cu")
-		(net 12)
-	)
-	(segment
-		(start 177.25 99.25)
-		(end 179.25 97.25)
-		(width 0.2)
-		(layer "B.Cu")
-		(net 12)
-	)
-	(segment
-		(start 191.7227 82.6277)
-		(end 191.7227 78.2473)
+		(start 184.35 102.1)
+		(end 182.75 100.5)
 		(width 0.2)
 		(layer "B.Cu")
@@
 	)
 	(segment
+		(start 191.7227 78.2473)
+		(end 191.93 78.04)
+		(width 0.2)
+		(layer "B.Cu")
+		(net 46)
+	)
+	(segment
 		(start 197.0209 96.2977)
 		(end 198.8842 94.4344)
@@
 		(polygon
 			(pts
-				(xy 100.75 76) (xy 101 105.5) (xy 222.25 105.5) (xy 222.25 76)
+				(xy 100.781346 76) (xy 101.031346 105.5) (xy 222.281346 105.5) (xy 222.281346 76)
 			)
 		)
