File: 26th_PCB_PitchSender.kicad_sch (KiCad schematic)
At the start: 9 parts, among them J1 Conn_01x04_Socket, J2 Conn_01x04_Pin, J3 Micro_SD_Card_Det1, J4 Conn_01x04_Socket, J5 Conn_01x04_Socket

Commit message: BMP追加
Parts:
- added D2, D3: LED, LED_THT:LED_D3.0mm, symbol Device:LED
- added J6: BMP390, Connector_PinHeader_2.54mm:PinHeader_1x04_P2.54mm_Vertical, symbol Connector:Conn_01x04_Socket
- added R2, R3: R, Resistor_THT:R_Axial_DIN0204_L3.6mm_D1.6mm_P5.08mm_Horizontal, symbol Device:R
- J1: value Conn_01x04_Socket -> vol
- J3: value Micro_SD_Card_Det1 -> microSD
- J5: value Conn_01x04_Socket -> BNO055
Connections:
- net +3V3: now also J6.1 (Pin_1)
- net GND: now also D2.1 (K), D3.1 (K), J6.2 (Pin_2)
- net SCL: now also J6.3 (Pin_3)
- net SDA: now also J6.4 (Pin_4)
- net at U1.J3_13 (IO4): now also R2.1
- net at U1.J3_16 (IO15): now also R3.1
- new net: D2.2 (A), R2.2
- new net: D3.2 (A), R3.2
- no-connect marks 33 -> 31
Other:
- note added: "BMP390"
